File: kicad/SIM900.sch (KiCad schematic (older format))
At the start: 9 parts

Commit message: z
Parts:
- removed J?: SIM_Card, symbol Connector:SIM_Card
- added D?: D_Schottky, symbol Device:D_Schottky
- added D? (x2): LED, symbol Device:LED
- added J?: SIM_Card, symbol jagKiCAD:SIM_Card
- added J?: Conn_Coaxial, symbol Connector:Conn_Coaxial
- added J?: Pin header, symbol Connector:Conn_01x02_Male
- added Q? (x4): Q_NPN_BEC, symbol Device:Q_NPN_BEC
- added R? (x5): R_Small, symbol Device:R_Small
- added R? (x4): 100k, symbol Device:R_Small
- added R? (x4): 4.7k, symbol Device:R_Small
- added R?: 220, symbol Device:R
- added R?: 200, symbol Device:R
- added U?: SP0505BA, symbol jagKiCAD:SMF05C
Connections:
- net +4V: now also R?.1, R?.1
- net GND: now also BT?.2 (-), U?.17 (GND), U?.18 (GND), U?.29 (GND), U?.39 (GND), U?.45 (GND), U?.46 (GND), U?.53 (GND), U?.54 (GND), U?.58 (GND), U?.59 (GND), U?.61 (GND), U?.62 (GND), U?.63 (GND), U?.64 (GND), U?.65 (GND), J?.2 (Ext), J?.5 (GND), Q?.2 (E), Q?.2 (E), Q?.2 (E), Q?.2 (E), R?.1, R?.1, R?.1, R?.1, U?.2
- net SIM900_RX: now also R?.2; no longer U?.10 (RXD)
- net SIM900_TX: now also R?.2; no longer U?.9 (TXD)
- net at U?.1 (PWRKEY): now also Q?.3 (C)
- net at U?.16 (~RESET~): now also Q?.3 (C)
- net at U?.26 (VRTC): now also D?.1 (K)
- net at U?.27 (DBG_TXD): now also J?.1 (Pin_1)
- net at U?.28 (DBG_RXD): now also J?.2 (Pin_2)
- net at U?.30 (SIM_VDD): now also J?.1 (VCC), U?.1
- net at U?.31 (SIM_DATA): now also R?.2
- net at U?.32 (SIM_CLK): now also R?.2
- net at U?.33 (SIM_RST): now also R?.2
- net NETLIGHT: now reaches U?.52 (NETLIGHT)
- net NETLIGHT: now also R?.2
- net at U?.60 (RF_ANT): now also J?.1 (In)
- net STATUS: now reaches U?.66 (STATUS)
- net STATUS: now also R?.2
- net at BT?.1 (+): now also D?.2 (A)
- new net: R?.1, U?.10 (RXD)
- new net: R?.1, U?.9 (TXD)
- new net: J?.7 (I/O), R?.1, U?.3
- new net: J?.3 (CLK), R?.1, U?.4
- new net: J?.2 (RST), R?.1, U?.5
- new net: Q?.1 (B), R?.1, R?.2 (x4)
- new net: D?.1 (K), Q?.3 (C) (x2)
- new net: D?.2 (A), R?.2 (x2)
- new net PWRKEY: R?.2
- new net RESET: R?.2
- no-connect marks 1 -> 34
Other:
- note added: "Debug"
- note added: "LEDs"
- note added: "SIM900 status LEDs"
- moved on the sheet: BT?, C?, U?
