File: kicad/relays.sch (KiCad schematic (older format))
At the start: 21 parts

Commit message: fg
Other:
- note added: "Double isolated"
- note added: "LV side"
- note added: "Mains side"
Changed lines of the file:
@@
 $Descr A4 11693 8268
 encoding utf-8
-Sheet 4 6
+Sheet 5 6
 Title "Estufes Saillagouse"
 Date "2019-12-30"
@@
 NoConn ~ 5450 1300
 NoConn ~ 5450 5700
+Wire Notes Line width 39
+	5350 7550 5350 850
+Wire Notes Line width 39
+	3450 7550 3450 850
+Text Notes 3700 750  0    118  ~ 0
+Double isolated
+Text Notes 2400 750  0    118  ~ 0
+LV side
+Text Notes 5650 750  0    118  ~ 0
+Mains side
 $EndSCHEMATC
